File: LucidDAC.kicad_pcb (KiCad board)
At the start: 2 copper layers, 62 x 26.2 mm, 48 parts, among them J1 J1, J2 USB_C_Receptacle_USB2.0_16P, J3 SJ-435107, SW1 MIC_GAIN, SW2 MIC_MUTE, U1 USBLC6-2SC6, U2 PCM2912APJTR, Y1 6MHz

Commit message: update pcb
Parts:
- removed C2, C3: 220uF, Capacitor_SMD:C_0805_2012Metric_Pad1.18x1.45mm_HandSolder
- added CE1: 220uF, EEEFK1A221XP:CAP_EEEFK1A221XP, F.Cu at (59.9, 37.3)
- added CE2: 220uF, EEEFK1A221XP:CAP_EEEFK1A221XP, F.Cu at (60.5, 23.4)
- moved C5 15.8 mm to (46.4, 36.6)
- moved J1 15.1 mm to (57.1, 31.9), turned to 90 degrees
- moved C4 13.6 mm to (46.4, 30.2)
- moved R5 12.0 mm to (48.3, 28.1)
- moved R8 11.0 mm to (49.4, 35.6), turned to 90 degrees
- moved C19 10.8 mm to (25.3, 35.8), turned to 90 degrees
- moved R7 9.60 mm to (49.4, 31.2), turned to -90 degrees
- moved C6 8.89 mm to (46.4, 32.3)
- moved C7 8.77 mm to (46.4, 34.5)
- moved MIC_GAIN 8.74 mm to (46.6, 24.9), turned to 180 degrees
- moved JP1 7.93 mm to (42.3, 24.2)
- moved R11 7.67 mm to (58.2, 42.2), turned to 180 degrees
- moved R9 7.56 mm to (42.3, 21.8), turned to 0 degrees
- moved R3 7.50 mm to (67.2, 23.4), turned to 0 degrees
- moved U2 6.96 mm to (38.7, 32.9)
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- renumbered SW1 to MIC_GAIN, SW2 to MIC_MUTE
Routing:
- net H_GND: track 134.8 -> 157.0 mm, vias 7 -> 6
- net MAMP: track 14.1 -> 23.7 mm, vias 0 -> 3
- net Net-(U2-MBIAS): track 13.9 -> 23.0 mm
- net XTO: track 26.9 -> 18.8 mm
- net VCCP: track 15.7 -> 8.22 mm
- net XTI: track 21.4 -> 14.0 mm
- net Net-(U2-VBUS): track 14.3 -> 8.09 mm
- net TRRS_RING_2: track 21.8 -> 15.9 mm
- net Net-(U2-VOUTR): track 24.0 -> 18.7 mm, vias 2 -> 0
- net Net-(U2-D+): track 9.46 -> 4.24 mm
- net Net-(U2-D-): track 9.38 -> 4.57 mm
- net Net-(U2-VOUTL): track 22.4 -> 18.0 mm, vias 3 -> 2
- net VBUS: track 30.2 -> 26.1 mm
- net D+: track 8.65 -> 4.60 mm
- net MMUTE: track 3.48 -> 7.31 mm
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